Commit message: Refactor robot description

File: rover_description/urdf/car.urdf.xacro (robot description, xacro)
@@ -40,16 +40,4 @@
   <xacro:property name="chassis_height" value="0.01"/>
   <xacro:property name="chassis_mass" value="2.788"/>
-  <!-- battery_dist is the distance between the inner edges of the
-       batteries. battery_comp_depth is the battery compartment depth.
-       battery_length is measured along the x axis, battery_width
-       along the y axis, and battery_height along the z axis. -->
-  <xacro:property name="battery_x_offset" value="0.055"/>
-  <xacro:property name="battery_dist" value="0.065"/>
-  <xacro:property name="battery_comp_depth" value="0.02"/>
-  <xacro:property name="battery_comp_angle" value="0.34906585"/>
-  <xacro:property name="battery_length" value="0.16"/>
-  <xacro:property name="battery_width" value="0.047"/>
-  <xacro:property name="battery_height" value="0.024"/>
-  <xacro:property name="battery_mass" value="0.5025"/>
   <!-- hub_dia and tire_dia are the diameters of the hub and tire,
        respectively. hex_hub_depth is the distance that the hex hub is
@@ -98,7 +86,4 @@
   <!-- ctrl_period is gazebo_ros_control's control period. Unit: hertz. -->
   <xacro:property name="ctrl_period" value="0.01"/>
-  <material name="battery_mat">
-    <color rgba="0 0 1 1"/>
-  </material>
   <material name="chassis_mat">
     <color rgba="0.5 0.5 0.5 1"/>
@@ -145,46 +130,4 @@
                     outer_rad * outer_rad) / 2}"/>
     </inertial>
-  </xacro:macro>
-  <!-- Battery -->
-  <xacro:macro name="battery" params="prefix reflect">
-    <joint name="chassis_to_${prefix}_battery" type="fixed">
-      <parent link="chassis"/>
-      <child link="${prefix}_battery_offset"/>
-      <origin xyz="${battery_x_offset - battery_length / 2}
-                   ${reflect * battery_dist / 2}
-                   0"
-              rpy="${reflect * battery_comp_angle} 0 0"/>
-    </joint>
-    <link name="${prefix}_battery_offset">
-      <xacro:null_inertial/>
-    </link>
-    <joint name="offset_to_${prefix}_battery" type="fixed">
-      <parent link="${prefix}_battery_offset"/>
-      <child link="${prefix}_battery"/>
-      <origin xyz="0
-                   ${reflect * battery_width / 2}
-                   ${(battery_height / 2) - battery_comp_depth}"/>
-    </joint>
-    <link name="${prefix}_battery">
-      <visual>
-        <geometry>
-          <box size="${battery_length} ${battery_width} ${battery_height}"/>
-        </geometry>
-        <material name="battery_mat"/>
-      </visual>
-      <collision>
-        <geometry>
-          <box size="${battery_length} ${battery_width} ${battery_height}"/>
-        </geometry>
-      </collision>
-      <xacro:solid_cuboid_inertial
-         width="${battery_length}" depth="${battery_width}"
-         height="${battery_height}" mass="${battery_mass}">
-        <origin/>
-      </xacro:solid_cuboid_inertial>
-    </link>
-    <gazebo reference="${prefix}_battery">
-      <material>Gazebo/Blue</material>
-    </gazebo>
   </xacro:macro>
   <!-- Shock absorber -->
@@ -336,5 +279,5 @@
     <origin xyz="${chassis_length /2 + 0.12} 0.0 0.0" rpy="0.0 0.0 0.0"/>
   </joint>
-    <joint name="imu_joint" type="fixed">
+  <joint name="imu_joint" type="fixed">
 		<axis xyz="1 0 0"/>
 		<origin xyz="0 0 0.19"/>
@@ -389,7 +332,4 @@
     <child link="chassis"/>
   </joint>
-  <!-- Batteries -->
-  <xacro:battery prefix="left" reflect="1"/>
-  <xacro:battery prefix="right" reflect="-1"/>
   <!-- Wheels -->
   <xacro:front_wheel lr_prefix="left" fr_prefix="front"
@@ -402,11 +342,5 @@
                     lr_reflect="-1" fr_reflect="-1"/>
   <gazebo>
-    <plugin name="gazebo_ros_control" filename="libgazebo_ros_control.so">
-      <!-- As of 10/7/13, setting controlPeriod to a value greater than
-           Gazebo's simulation period prevents the shock absorbers from
-           working.
-      <controlPeriod>${ctrl_period}</controlPeriod>
-      -->
-    </plugin>
+    <plugin name="gazebo_ros_control" filename="libgazebo_ros_control.so" />
   </gazebo>
   <!-- Depth sensor -->
@@ -440,5 +374,5 @@
   <plugin name="magnetic_sim" filename="libhector_gazebo_ros_magnetic.so">
     <alwaysOn>true</alwaysOn>
-    <topicName>magnetic/raw</topicName>
+    <topicName>magnetic/data</topicName>
     <updateRate>100.0</updateRate>
     <bodyName>imu_link</bodyName>

Commit message: Update rover to 6 wheeled rocker-bogie

File: rover_description/urdf/car.urdf.xacro (robot description, xacro)
@@ -1,43 +1,19 @@
 <?xml version="1.0"?>
-<!-- car.urdf.xacro
-This file defines a model of a RC Car augmented with sensors
-It is based on the Traxxas(R) E-Maxx(R) #3905 RC (Radio Controlled)
-truck model:
-Here below are the description given for the em_3905 model:
-Lengths are measured in meters, angles are measured in radians, and masses are
-measured in kilograms. All of these values are approximations.
-To work with Gazebo, each link must have an inertial element, even if
-the link only serves to connect two joints. To be visible in Gazebo, a link
-must have a collision element. Furthermore, the link must have a Gazebo
-material.
-Traxxas(R), E-Maxx(R), and Titan(R) are registered trademarks of Traxxas
-Management, LLC. em_3905.urdf.xacro was independently created by Wunderkammer
-Laboratory, and neither em_3905.urdf.xacro nor Wunderkammer Laboratory is
-affiliated with, sponsored by, approved by, or endorsed by Traxxas Management,
-LLC. Mabuchi Motor(R) is a registered trademark of Mabuchi Motor Co., Ltd.
-Corporation Japan. All other trademarks and service marks are the property of
-their respective owners.
-Copyright (c) 2011-2013 Wunderkammer Laboratory
-Licensed under the Apache License, Version 2.0 (the "License");
-you may not use this file except in compliance with the License.
-You may obtain a copy of the License at
-  http://www.apache.org/licenses/LICENSE-2.0
-Unless required by applicable law or agreed to in writing, software
-distributed under the License is distributed on an "AS IS" BASIS,
-WITHOUT WARRANTIES OR CONDITIONS OF ANY KIND, either express or implied.
-See the License for the specific language governing permissions and
-limitations under the License.
--->
 <robot name="rover" xmlns:xacro="http://www.ros.org/wiki/xacro">
   <!-- Degree-to-radian conversions -->
   <xacro:property name="degrees_45" value="0.785398163"/>
   <xacro:property name="degrees_90" value="1.57079633"/>
-  <!-- chassis_length is measured along the x axis, chassis_width
-       along the y axis, and chassis_height along the z axis. -->
-  <!--xacro:property name="chassis_length" value="0.258"/-->
-  <xacro:property name="chassis_length" value="0.35"/>
-  <xacro:property name="chassis_width" value="0.168"/>
-  <xacro:property name="chassis_height" value="0.01"/>
-  <xacro:property name="chassis_mass" value="2.788"/>
+  <!-- body_length is measured along the x axis, body_width
+       along the y axis, and body_height along the z axis. -->
+  <xacro:property name="body_length"    value="0.350"/>
+  <xacro:property name="body_width"     value="0.200"/>
+  <xacro:property name="body_height"    value="0.100"/>
+  <xacro:property name="body_mass"      value="2.788"/>
+  <xacro:property name="body_clearance" value="0.200"/>
+  <xacro:property name="wheelbase_rocker" value="0.350"/>
+  <xacro:property name="wheelbase_bogie"  value="0.200"/>
+  <xacro:property name="x_center_rocker"  value="0.000"/>
+  <xacro:property name="x_center_bogie"   value="0.150"/>
+  <xacro:property name="track"            value="0.350"/>
   <!-- hub_dia and tire_dia are the diameters of the hub and tire,
        respectively. hex_hub_depth is the distance that the hex hub is
@@ -45,24 +21,8 @@
        is a "zero offset" wheel. hex_hub_depth = tire_width / 2 -
        axle_length. -->
-  <xacro:property name="hub_dia" value="0.09652"/>
-  <xacro:property name="tire_dia" value="0.14605"/>
-  <xacro:property name="tire_width" value="0.0889"/>
-  <xacro:property name="hex_hub_depth" value="0.01445"/>
-  <xacro:property name="wheel_mass" value="0.29"/>
-  <!-- hex_hub_dist is the distance between left and right hex hubs when
-       the shock absorbers are fully extended. axle_length is the distance
-       from a U joint to the corresponding hex hub. wheel_travel is the
-       vertical wheel travel. -->
-  <xacro:property name="wheelbase" value="0.335"/>
-  <xacro:property name="hex_hub_dist" value="0.365"/>
-  <xacro:property name="axle_length" value="0.03"/>
-  <xacro:property name="wheel_travel" value="0.084"/>
-  <xacro:property name="shock_z_offset" value="0.0655"/>
-  <!-- shock_eff_limit is 2 * ((shock_stroke / 2) * shock_spring_constant) N.
-       shock_stroke is 0.028575 meters. shock_spring_constant, an approximation
-       of a Traxxas Ultra Shock shock absorber spring's constant, is
-       437.817 N/m. -->
-  <xacro:property name="shock_eff_limit" value="12.5106"/>
-  <xacro:property name="shock_vel_limit" value="1000"/>
+  <xacro:property name="hub_dia"       value="0.100"/>
+  <xacro:property name="tire_dia"      value="0.115"/>
+  <xacro:property name="tire_width"    value="0.075"/>
+  <xacro:property name="wheel_mass"    value="0.200"/>
   <!-- The specifications for a Titan(R) 550 motor could not be found, so the
        stall torque of a Mabuchi Motor(R) RS-550VC-7525 motor was used instead.
@@ -79,12 +39,5 @@
   <xacro:property name="axle_eff_limit" value="5.12766"/>
   <xacro:property name="axle_vel_limit" value="244.8696"/>
-  <!-- These constants are used to simulate a Traxxas 2056 servo operated at
-       6 V. servo_stall_torque is measured in N m. servo_no_load_speed is
-       measured in rad/s. -->
-  <xacro:property name="servo_stall_torque" value="0.5649"/>
-  <xacro:property name="servo_no_load_speed" value="4.553"/>
-  <!-- ctrl_period is gazebo_ros_control's control period. Unit: hertz. -->
-  <xacro:property name="ctrl_period" value="0.01"/>
-  <material name="chassis_mat">
+  <material name="body_mat">
     <color rgba="0.5 0.5 0.5 1"/>
   </material>
@@ -131,39 +84,13 @@
     </inertial>
   </xacro:macro>
-  <!-- Shock absorber -->
-  <xacro:macro name="shock"
-               params="lr_prefix fr_prefix lr_reflect fr_reflect child">
-    <joint name="${lr_prefix}_${fr_prefix}_shock" type="prismatic">
-      <parent link="chassis"/>
-      <child link="${child}"/>
-      <origin xyz="${fr_reflect * wheelbase / 2}
-                   ${lr_reflect * ((hex_hub_dist / 2) - axle_length)}
-                   ${(wheel_travel / 2) - shock_z_offset}"/>
-      <axis xyz="0 0 -1"/>
-      <limit lower="${-wheel_travel / 2}" upper="${wheel_travel / 2}"
-             effort="${shock_eff_limit}" velocity="${shock_vel_limit}"/>
-    </joint>
-    <transmission name="${lr_prefix}_${fr_prefix}_shock_trans">
-      <type>transmission_interface/SimpleTransmission</type>
-      <joint name="${lr_prefix}_${fr_prefix}_shock">
-        <hardwareInterface>EffortJointInterface</hardwareInterface>
-      </joint>
-      <actuator name="${lr_prefix}_${fr_prefix}_shock_act">
-        <hardwareInterface>EffortJointInterface</hardwareInterface>
-        <mechanicalReduction>1</mechanicalReduction>
-      </actuator>
-    </transmission>
-  </xacro:macro>
   <!-- The "wheel" macro defines an axle carrier, axle, and wheel. -->
-  <xacro:macro name="wheel" params="lr_prefix fr_prefix lr_reflect">
-    <link name="${lr_prefix}_${fr_prefix}_axle_carrier">
-      <xacro:null_inertial/>
-    </link>
-    <!-- The left and right axles have the same axis so that identical
-         rotation values cause the wheels to rotate in the same direction. -->
+  <xacro:macro name="wheel" params="lr_prefix fr_prefix lr_pos fr_pos">
     <joint name="${lr_prefix}_${fr_prefix}_axle" type="continuous">
-      <parent link="${lr_prefix}_${fr_prefix}_axle_carrier"/>
+      <parent link="base_link"/>
       <child link="${lr_prefix}_${fr_prefix}_wheel"/>
-      <origin rpy="${degrees_90} 0 0"/>
+      <origin xyz="${fr_pos}
+                   ${lr_pos}
+                   ${- body_clearance}"
+              rpy="${degrees_90} 0 0"/>
       <axis xyz="0 0 -1"/>
       <limit effort="${axle_eff_limit}" velocity="${axle_vel_limit}"/>
@@ -181,8 +108,5 @@
     <link name="${lr_prefix}_${fr_prefix}_wheel">
       <visual>
-        <origin xyz="0
-                     ${lr_reflect * (axle_length - (tire_width /
-                     2 - hex_hub_depth))}
-                     0"/>
+        <origin xyz="0 0 0"/>
         <geometry>
           <cylinder radius="${tire_dia / 2}" length="${tire_width}"/>
@@ -191,8 +115,5 @@
       </visual>
       <collision>
-        <origin xyz="0
-                     ${lr_reflect * (axle_length - (tire_width /
-                     2 - hex_hub_depth))}
-                     0"/>
+        <origin xyz="0 0 0"/>
         <geometry>
           <cylinder radius="${tire_dia / 2}" length="${tire_width}"/>
@@ -207,42 +128,4 @@
     </gazebo>
   </xacro:macro>
-  <!-- Front wheel -->
-  <xacro:macro name="front_wheel"
-               params="lr_prefix fr_prefix lr_reflect fr_reflect">
-    <xacro:shock lr_prefix="${lr_prefix}" fr_prefix="${fr_prefix}"
-                 lr_reflect="${lr_reflect}" fr_reflect="${fr_reflect}"
-                 child="${lr_prefix}_steering_link"/>
-    <link name="${lr_prefix}_steering_link">
-      <xacro:null_inertial/>
-    </link>
-    <joint name="${lr_prefix}_steering_joint" type="revolute">
-      <parent link="${lr_prefix}_steering_link"/>
-      <child link="${lr_prefix}_${fr_prefix}_axle_carrier"/>
-      <axis xyz="0 0 1"/>
-      <limit lower="${-degrees_45}" upper="${degrees_45}"
-             effort="${servo_stall_torque}" velocity="${servo_no_load_speed}"/>
-    </joint>
-    <transmission name="${lr_prefix}_steering_trans">
-      <type>transmission_interface/SimpleTransmission</type>
-      <joint name="${lr_prefix}_steering_joint">
-        <hardwareInterface>EffortJointInterface</hardwareInterface>
-      </joint>
-      <actuator name="${lr_prefix}_steering_act">
-        <hardwareInterface>EffortJointInterface</hardwareInterface>
-        <mechanicalReduction>1</mechanicalReduction>
-      </actuator>
-    </transmission>
-    <xacro:wheel lr_prefix="${lr_prefix}" fr_prefix="${fr_prefix}"
-                 lr_reflect="${lr_reflect}"/>
-  </xacro:macro>
-  <!-- Rear wheel -->
-  <xacro:macro name="rear_wheel"
-               params="lr_prefix fr_prefix lr_reflect fr_reflect">
-    <xacro:shock lr_prefix="${lr_prefix}" fr_prefix="${fr_prefix}"
-                 lr_reflect="${lr_reflect}" fr_reflect="${fr_reflect}"
-                 child="${lr_prefix}_${fr_prefix}_axle_carrier"/>
-    <xacro:wheel lr_prefix="${lr_prefix}" fr_prefix="${fr_prefix}"
-                 lr_reflect="${lr_reflect}"/>
-  </xacro:macro>
   <!-- base_link must have geometry so that its axes can be displayed in
        rviz. -->
@@ -252,5 +135,5 @@
         <box size="0.05 0.05 0.01"/>
       </geometry>
-      <material name="chassis_mat"/>
+      <material name="body_mat"/>
     </visual>
   </link>
@@ -258,28 +141,7 @@
     <material>Gazebo/Green</material>
   </gazebo>
-  <link name="bumper_link">
-	    <visual>
-	        <geometry>
-	            <box size="0.01 0.3 0.01"/>
-	        </geometry>
-	    </visual>
-	    <collision>
-	        <!-- origin is relative -->
-	        <geometry>
-	            <box size="0.01 0.3 0.01"/>
-	        </geometry>
-	    </collision>
-	</link>
-	<gazebo reference="bumper_link">
-  	<material>Gazebo/Black</material>
-  </gazebo>
-  <joint name="baselink_to_bumper" type="fixed">
-    <parent link="base_link"/>
-    <child link="bumper_link"/>
-    <origin xyz="${chassis_length /2 + 0.12} 0.0 0.0" rpy="0.0 0.0 0.0"/>
-  </joint>
   <joint name="imu_joint" type="fixed">
 		<axis xyz="1 0 0"/>
-		<origin xyz="0 0 0.19"/>
+		<origin xyz="0 0 0.05"/>
 		<parent link="base_link"/>
 		<child link="imu_link"/>
@@ -304,41 +166,57 @@
 	  </collision>
 	</link>
-  <!-- Chassis -->
-  <link name="chassis">
+  <!-- body -->
+  <link name="body">
     <visual>
-      <origin xyz="0 0 ${-chassis_height / 2}"/>
+      <origin xyz="0 0 ${-body_height / 2}"/>
       <geometry>
-        <box size="${chassis_length} ${chassis_width} ${chassis_height}"/>
+        <box size="${body_length} ${body_width} ${body_height}"/>
       </geometry>
-      <material name="chassis_mat"/>
+      <material name="body_mat"/>
     </visual>
     <collision>
-      <origin xyz="0 0 ${-chassis_height / 2}"/>
+      <origin xyz="0 0 ${-body_height / 2}"/>
       <geometry>
-        <box size="${chassis_length} ${chassis_width} ${chassis_height}"/>
+        <box size="${body_length} ${body_width} ${body_height}"/>
       </geometry>
     </collision>
     <xacro:solid_cuboid_inertial
-        width="${chassis_length}" depth="${chassis_width}"
-        height="${chassis_height}" mass="${chassis_mass}">
-      <origin xyz="0 0 ${-chassis_height / 2}"/>
+        width="${body_length}" depth="${body_width}"
+        height="${body_height}" mass="${body_mass}">
+      <origin xyz="0 0 ${-body_height / 2}"/>
     </xacro:solid_cuboid_inertial>
   </link>
-  <gazebo reference="chassis">
+  <gazebo reference="body">
     <material>Gazebo/Grey</material>
   </gazebo>
   <joint name="base_link_to_chasis" type="fixed">
     <parent link="base_link"/>
-    <child link="chassis"/>
+    <child link="body"/>
   </joint>
   <!-- Wheels -->
-  <xacro:front_wheel lr_prefix="left" fr_prefix="front"
-                     lr_reflect="1" fr_reflect="1"/>
-  <xacro:front_wheel lr_prefix="right" fr_prefix="front"
-                     lr_reflect="-1" fr_reflect="1"/>
-  <xacro:rear_wheel lr_prefix="left" fr_prefix="rear"
-                    lr_reflect="1" fr_reflect="-1"/>
-  <xacro:rear_wheel lr_prefix="right" fr_prefix="rear"
-                    lr_reflect="-1" fr_reflect="-1"/>
+  <xacro:wheel lr_prefix="left_bogie" fr_prefix="front"
+               lr_pos="${track / 2}"
+               fr_pos="${x_center_bogie + wheelbase_bogie / 2}"
+               />
+  <xacro:wheel lr_prefix="left_bogie" fr_prefix="rear"
+               lr_pos="${track / 2}"
+               fr_pos="${x_center_bogie - wheelbase_bogie / 2}"
+               />
+  <xacro:wheel lr_prefix="left_rocker" fr_prefix="rear"
+               lr_pos="${track / 2}"
+               fr_pos="${x_center_rocker - wheelbase_rocker / 2}"
+               />
+  <xacro:wheel lr_prefix="right_bogie" fr_prefix="front"
+               lr_pos="${- track / 2}"
+               fr_pos="${x_center_bogie + wheelbase_bogie / 2}"
+               />
+  <xacro:wheel lr_prefix="right_bogie" fr_prefix="rear"
+               lr_pos="${- track / 2}"
+               fr_pos="${x_center_bogie - wheelbase_bogie / 2}"
+               />
+  <xacro:wheel lr_prefix="right_rocker" fr_prefix="rear"
+               lr_pos="${- track / 2}"
+               fr_pos="${x_center_rocker - wheelbase_rocker / 2}"
+               />
   <gazebo>
     <plugin name="gazebo_ros_control" filename="libgazebo_ros_control.so" />

Commit message: Use skid steer control on rocker-bogie rover

File: rover_description/urdf/car.urdf.xacro (robot description, xacro)
@@ -6,8 +6,8 @@
   <!-- body_length is measured along the x axis, body_width
        along the y axis, and body_height along the z axis. -->
-  <xacro:property name="body_length"    value="0.350"/>
-  <xacro:property name="body_width"     value="0.200"/>
-  <xacro:property name="body_height"    value="0.100"/>
-  <xacro:property name="body_mass"      value="2.788"/>
+  <xacro:property name="body_length"    value="0.300"/>
+  <xacro:property name="body_width"     value="0.250"/>
+  <xacro:property name="body_height"    value="0.050"/>
+  <xacro:property name="body_mass"      value="3.000"/>
   <xacro:property name="body_clearance" value="0.200"/>
   <xacro:property name="wheelbase_rocker" value="0.350"/>
@@ -15,5 +15,5 @@
   <xacro:property name="x_center_rocker"  value="0.000"/>
   <xacro:property name="x_center_bogie"   value="0.150"/>
-  <xacro:property name="track"            value="0.350"/>
+  <xacro:property name="track"            value="0.400"/>
   <!-- hub_dia and tire_dia are the diameters of the hub and tire,
        respectively. hex_hub_depth is the distance that the hex hub is
@@ -99,8 +99,8 @@
       <type>transmission_interface/SimpleTransmission</type>
       <joint name="${lr_prefix}_${fr_prefix}_axle">
-        <hardwareInterface>EffortJointInterface</hardwareInterface>
+        <hardwareInterface>VelocityJointInterface</hardwareInterface>
       </joint>
       <actuator name="${lr_prefix}_${fr_prefix}_axle_act">
-        <hardwareInterface>EffortJointInterface</hardwareInterface>
+        <hardwareInterface>VelocityJointInterface</hardwareInterface>
         <mechanicalReduction>1</mechanicalReduction>
       </actuator>
@@ -225,5 +225,5 @@
   <xacro:include filename="$(find rover_description)/urdf/depth_sensor.urdf.xacro" />
   <xacro:depth_sensor name="camera" parent="base_link">
-    <origin xyz="0.15 0.0 0.05" rpy="0 0 0"/>
+    <origin xyz="${body_length / 2 + 0.05} 0.0 ${- body_height / 4}" rpy="0 0 0"/>
   </xacro:depth_sensor>
   <!-- IMU sensor-->
